Commit message: add helpers to calculate distance and apply rotation angles

File: intraining_specimen/r_9be70e16-e36e-4124-8bfa-6fae9efd751d.urdf (robot description, URDF)
Before this commit: robot robot, 18 links, 17 joints
Links:
- removed link link_0_0
- removed link link_0_1
- removed link link_0_2
- removed link link_0_3
- removed link link_0_4
- removed link link_0_5
- removed link link_0_6
- removed link link_0_7
- removed link link_0_8
- removed link link_1_0
- removed link link_1_1
- removed link link_1_2
- removed link link_1_3
- added link finger_link_0_0, mass 0.025; collision box size=0.034 0.032 0.078; visual box size=0.034 0.032 0.078
- added link finger_link_0_1, mass 0.034; collision box size=0.05 0.038 0.06; visual box size=0.05 0.038 0.06
- added link finger_link_0_2, mass 0.003; collision box size=0.021 0.022 0.025; visual box size=0.021 0.022 0.025
- added link finger_link_0_3, mass 0.008; collision box size=0.028 0.017 0.057; visual box size=0.028 0.017 0.057
- added link finger_link_0_4, mass 0.01; collision box size=0.023 0.044 0.032; visual box size=0.023 0.044 0.032
- added link finger_link_0_5, mass 0.007; collision box size=0.012 0.034 0.055; visual box size=0.012 0.034 0.055
- added link finger_link_0_6, mass 0.01; collision box size=0.035 0.038 0.025; visual box size=0.035 0.038 0.025
- added link finger_link_0_7, mass 0.005; collision box size=0.04 0.017 0.023; visual box size=0.04 0.017 0.023
- added link finger_link_0_8, mass 0.017; collision box size=0.022 0.034 0.074; visual box size=0.022 0.034 0.074
- added link finger_link_1_0, mass 0.01; collision box size=0.049 0.022 0.032; visual box size=0.049 0.022 0.032
- added link finger_link_1_1, mass 0.012; collision box size=0.027 0.018 0.081; visual box size=0.027 0.018 0.081
- added link finger_link_1_2, mass 0.007; collision box size=0.014 0.045 0.039; visual box size=0.014 0.045 0.039
- added link finger_link_1_3, mass 0.008; collision box size=0.025 0.023 0.047; visual box size=0.025 0.023 0.047
Joints:
- removed joint joint_link_0_0_to_link_0_1
- removed joint joint_link_0_1_to_link_0_2
- removed joint joint_link_0_2_to_link_0_3
- removed joint joint_link_0_3_to_link_0_4
- removed joint joint_link_0_4_to_link_0_5
- removed joint joint_link_0_5_to_link_0_6
- removed joint joint_link_0_6_to_link_0_7
- removed joint joint_link_0_7_to_link_0_8
- removed joint joint_link_1_0_to_link_1_1
- removed joint joint_link_1_1_to_link_1_2
- removed joint joint_link_1_2_to_link_1_3
- removed joint joint_palm_link_to_link_0_0
- removed joint joint_palm_link_to_link_1_0
- added joint joint_finger_link_0_0_to_finger_link_0_1: type revolute, parent finger_link_0_0, child finger_link_0_1, origin xyz=0.0 0.0 0.078 rpy=0 0 0, axis 0.811 0.108 0.521, limit lower=-3.142 upper=3.142 effort=10 velocity=10
- added joint joint_finger_link_0_1_to_finger_link_0_2: type revolute, parent finger_link_0_1, child finger_link_0_2, origin xyz=0.0 0.0 0.06 rpy=0 0 0, axis 0.904 0.073 0.923, limit lower=-3.142 upper=3.142 effort=10 velocity=10
- added joint joint_finger_link_0_2_to_finger_link_0_3: type revolute, parent finger_link_0_2, child finger_link_0_3, origin xyz=0.0 0.0 0.025 rpy=0 0 0, axis 0.7 0.169 0.557, limit lower=-3.142 upper=3.142 effort=10 velocity=10
- added joint joint_finger_link_0_3_to_finger_link_0_4: type revolute, parent finger_link_0_3, child finger_link_0_4, origin xyz=0.0 0.0 0.057 rpy=0 0 0, axis 0.898 0.816 0.407, limit lower=-3.142 upper=3.142 effort=10 velocity=10
- added joint joint_finger_link_0_4_to_finger_link_0_5: type revolute, parent finger_link_0_4, child finger_link_0_5, origin xyz=0.0 0.0 0.032 rpy=0 0 0, axis 0.785 0.339 0.425, limit lower=-3.142 upper=3.142 effort=10 velocity=10
- added joint joint_finger_link_0_5_to_finger_link_0_6: type revolute, parent finger_link_0_5, child finger_link_0_6, origin xyz=0.0 0.0 0.055 rpy=0 0 0, axis 0.419 0.282 0.844, limit lower=-3.142 upper=3.142 effort=10 velocity=10
- added joint joint_finger_link_0_6_to_finger_link_0_7: type revolute, parent finger_link_0_6, child finger_link_0_7, origin xyz=0.0 0.0 0.025 rpy=0 0 0, axis 0.996 0.958 0.288, limit lower=-3.142 upper=3.142 effort=10 velocity=10
- added joint joint_finger_link_0_7_to_finger_link_0_8: type revolute, parent finger_link_0_7, child finger_link_0_8, origin xyz=0.0 0.0 0.023 rpy=0 0 0, axis 0.706 0.774 0.224, limit lower=-3.142 upper=3.142 effort=10 velocity=10
- added joint joint_finger_link_1_0_to_finger_link_1_1: type revolute, parent finger_link_1_0, child finger_link_1_1, origin xyz=0.0 0.0 0.032 rpy=0 0 0, axis 0.467 0.863 0.894, limit lower=-3.142 upper=3.142 effort=10 velocity=10
- added joint joint_finger_link_1_1_to_finger_link_1_2: type revolute, parent finger_link_1_1, child finger_link_1_2, origin xyz=0.0 0.0 0.081 rpy=0 0 0, axis 0.341 0.41 0.322, limit lower=-3.142 upper=3.142 effort=10 velocity=10
- added joint joint_finger_link_1_2_to_finger_link_1_3: type revolute, parent finger_link_1_2, child finger_link_1_3, origin xyz=0.0 0.0 0.039 rpy=0 0 0, axis 0.994 0.563 0.56, limit lower=-3.142 upper=3.142 effort=10 velocity=10
- added joint joint_palm_link_to_finger_link_0_0: type revolute, parent palm_link, child finger_link_0_0, origin xyz=-0.086 0.125 0.1 rpy=0 0 0, axis 0.404 0.77 0.32, limit lower=-3.142 upper=3.142 effort=10 velocity=10
- added joint joint_palm_link_to_finger_link_1_0: type revolute, parent palm_link, child finger_link_1_0, origin xyz=-0.125 0.02 0.1 rpy=0 0 0, axis 0.458 0.132 0.81, limit lower=-3.142 upper=3.142 effort=10 velocity=10
- joint arm_joint: type revolute -> fixed
- joint support_joint: type continuous -> fixed
