Commit message: start adding modification so the specimen evolve better

File: objects/sphere_small.urdf (robot description, URDF)
Before this commit: robot sphere, 1 links, 0 joints
Links:
- link sphere: geometry collision sphere radius=0.01; visual sphere radius=0.01

File: robot_hand_test.urdf (robot description, URDF)
Before this commit: robot robot, 8 links, 7 joints
Links:
- removed link finger_link_0_0
- removed link finger_link_0_1
- removed link finger_link_0_2
Joints:
- removed joint finger_joint_finger_link_0_0_to_finger_link_0_1
- removed joint finger_joint_finger_link_0_1_to_finger_link_0_2
- removed joint finger_joint_palm_link_to_finger_link_0_0
