Commit message: add move fingers and move arm functionalities to specimen, some random specimen actually picking up the object

File: objects/cube.urdf (robot description, URDF)
Before this commit: robot cube, 1 links, 0 joints
Links:
- link cube: mass 10 -> 0.1

Commit message: modify distance calulation

File: objects/cube.urdf (robot description, URDF)
Before this commit: robot cube, 1 links, 0 joints
Links:
- link cube: mass 0.1 -> 0.01

File: objects/cylinder.urdf (robot description, URDF)
Before this commit: robot sphere, 1 links, 0 joints
Links:
- link sphere: mass 10 -> 0.01; geometry collision cylinder length=0.2 radius=0.1; visual cylinder length=0.2 radius=0.1

File: objects/sphere.urdf (robot description, URDF)
Before this commit: robot sphere, 1 links, 0 joints
Links:
- link sphere: mass 10 -> 0.01

File: objects/sphere_small.urdf (robot description, URDF)
Before this commit: robot sphere, 1 links, 0 joints
Links:
- link sphere: mass 10 -> 0.001
