Commit message: fix bug in brain mutation, and table moving

File: objects/table.urdf (robot description, URDF)
Before this commit: robot table, 2 links, 1 joints
Joints:
- joint table_joint: axis 0 1 0 -> (none); limit lower=0.0 upper=100.0 effort=10.0 velocity=10.0 -> (none); type prismatic -> fixed
