Commit message: evolve fit and add test objects

File: assets/misc/sphere_small.urdf (robot description, URDF)
Before this commit: robot sphere, 1 links, 0 joints
Links:
- link sphere: geometry collision sphere radius=0.1; visual sphere radius=0.1

File: assets/objects/cone.urdf (robot description, URDF)
Before this commit: robot cone, 1 links, 0 joints
Links:
- link cone: geometry collision mesh filename=cone.stl scale=1.2 1.2 1.2; visual mesh filename=cone.stl scale=1.2 1.2 1.2

File: assets/robot_arm/robot_arm copy.urdf (robot description, URDF)
Before this commit: robot robot_arm, 4 links, 3 joints
Links:
- added link finger_link_1, mass 1; collision cylinder length=0.25 radius=0.05; visual cylinder length=0.25 radius=0.05
- added link finger_link_2, mass 1; collision cylinder length=0.25 radius=0.05; visual cylinder length=0.25 radius=0.05
Joints:
- added joint finger_joint_1: type revolute, parent palm_link, child finger_link_1, origin xyz=-0.354 0.354 0 rpy=0 0 0, axis -1 -1 0, limit lower=-3.14 upper=3.14 effort=1.0 velocity=1.0
- added joint finger_joint_2: type fixed, parent finger_link_1, child finger_link_2, origin xyz=0 0 -0.25 rpy=0 0 0
- joint forearm_joint: origin xyz=0 0.75 3 rpy=0 -0.7854 0 -> xyz=0 0.75 3 rpy=0 0 0
